File: practicas/ELTEL/Q1/Practica1/Practica1Preg5/Practica1Preg5.sch (KiCad schematic (older format))
At the start: 4 parts

Commit message: Update
Parts:
- added BT2: 5, symbol Device:Battery_Cell
- added MES?: Amperemeter_DC, symbol Device:Amperemeter_DC
- added Re: 2000, symbol Device:R
- renumbered BT! to BT1
Connections:
- wire segments 7 -> 13
Other:
- moved on the sheet: BT1, MES?, R1, R2
Changed lines of the file:
@@
 $EndDescr
 Wire Wire Line
-	2150 1150 1950 1150
+	2136 640  1936 640
 $Comp
 L Device:Amperemeter_DC MES?
 U 1 1 5F7E3B06
-P 3050 1450
-F 0 "MES?" H 3203 1496 50  0000 L CNN
-F 1 "Amperemeter_DC" H 3203 1405 50  0000 L CNN
-F 2 "" V 3050 1550 50  0001 C CNN
-F 3 "~" V 3050 1550 50  0001 C CNN
-	1    3050 1450
+P 3036 940
+F 0 "MES?" H 3189 986 50  0000 L CNN
+F 1 "Amperemeter_DC" H 3189 895 50  0000 L CNN
+F 2 "" V 3036 1040 50  0001 C CNN
+F 3 "~" V 3036 1040 50  0001 C CNN
+	1    3036 940
 	1    0    0    -1
 $EndComp
@@
 L Device:R R2
 U 1 1 5F7E8191
-P 2750 1150
-F 0 "R2" V 2543 1150 50  0000 C CNN
-F 1 "1000" V 2634 1150 50  0000 C CNN
-F 2 "" V 2680 1150 50  0001 C CNN
-F 3 "~" H 2750 1150 50  0001 C CNN
-	1    2750 1150
+P 2736 640
+F 0 "R2" V 2529 640 50  0000 C CNN
+F 1 "1000" V 2620 640 50  0000 C CNN
+F 2 "" V 2666 640 50  0001 C CNN
+F 3 "~" H 2736 640 50  0001 C CNN
+	1    2736 640
 	0    1    1    0
 $EndComp
 Wire Wire Line
-	2450 1150 2600 1150
+	2436 640  2586 640
 Wire Wire Line
-	2900 1150 3050 1150
+	2886 640  3036 640
 Wire Wire Line
-	3050 1150 3050 1250
+	3036 640  3036 740
 $Comp
 L Device:R R1
 U 1 1 5F7E09EE
-P 2300 1150
-F 0 "R1" V 2093 1150 50  0000 C CNN
-F 1 "1000" V 2184 1150 50  0000 C CNN
-F 2 "" V 2230 1150 50  0001 C CNN
-F 3 "~" H 2300 1150 50  0001 C CNN
-	1    2300 1150
+P 2286 640
+F 0 "R1" V 2079 640 50  0000 C CNN
+F 1 "1000" V 2170 640 50  0000 C CNN
+F 2 "" V 2216 640 50  0001 C CNN
+F 3 "~" H 2286 640 50  0001 C CNN
+	1    2286 640
 	0    1    1    0
 $EndComp
 $Comp
-L Device:Battery_Cell BT!
+L Device:Battery_Cell BT1
 U 1 1 5F7EA385
-P 1950 1500
-F 0 "BT!" H 2068 1596 50  0000 L CNN
-F 1 "5" H 2068 1505 50  0000 L CNN
-F 2 "" V 1950 1560 50  0001 C CNN
-F 3 "~" V 1950 1560 50  0001 C CNN
-	1    1950 1500
+P 1936 990
+F 0 "BT1" H 2054 1086 50  0000 L CNN
+F 1 "5" H 2054 995 50  0000 L CNN
+F 2 "" V 1936 1050 50  0001 C CNN
+F 3 "~" V 1936 1050 50  0001 C CNN
+	1    1936 990
 	1    0    0    -1
 $EndComp
 Wire Wire Line
-	1950 1150 1950 1300
+	1936 640  1936 790
 Wire Wire Line
-	1950 1600 1950 1650
+	1936 1090 1936 1140
 Wire Wire Line
-	1950 1650 3050 1650
+	1936 1140 3036 1140
+$Comp
+L Device:Amperemeter_DC MES?
+U 1 1 5F7EEA61
+P 3021 1845
+F 0 "MES?" H 3174 1891 50  0000 L CNN
+F 1 "Amperemeter_DC" H 3174 1800 50  0000 L CNN
+F 2 "" V 3021 1945 50  0001 C CNN
+F 3 "~" V 3021 1945 50  0001 C CNN
+	1    3021 1845
+	1    0    0    -1
+$EndComp
+$Comp
+L Device:Battery_Cell BT2
+U 1 1 5F7EEAB0
+P 1921 1895
+F 0 "BT2" H 2039 1991 50  0000 L CNN
+F 1 "5" H 2039 1900 50  0000 L CNN
+F 2 "" V 1921 1955 50  0001 C CNN
+F 3 "~" V 1921 1955 50  0001 C CNN
+	1    1921 1895
+	1    0    0    -1
+$EndComp
+Wire Wire Line
+	1921 1995 1921 2045
+Wire Wire Line
+	1921 2045 3021 2045
+$Comp
+L Device:R Re
+U 1 1 5F7EFB71
+P 2494 1561
+F 0 "Re" V 2287 1561 50  0000 C CNN
+F 1 "2000" V 2378 1561 50  0000 C CNN
+F 2 "" V 2424 1561 50  0001 C CNN
+F 3 "~" H 2494 1561 50  0001 C CNN
+	1    2494 1561
+	0    1    1    0
+$EndComp
+Wire Wire Line
+	2645 1562 3023 1562
+Wire Wire Line
+	3023 1562 3023 1647
+Wire Wire Line
+	2347 1556 1920 1556
+Wire Wire Line
+	1920 1556 1920 1696
 $EndSCHEMATC
